File: hardware/VVVC_UserPort_Audio/VVVC_UserPort_Audio.kicad_pcb (KiCad board)
At the start: 2 copper layers, 100 x 80 mm, 22 parts, among them J1 VIC-20 USER PORT, J2 3.5mm TRS, J3 RCA IN L/R, J4 RCA OUT L/R, J5 5V DC IN, U2 NJM4556D / OPA1678

Commit message: Power carrier from ESP32 USB 5V
Parts:
- removed F1: PTC 1A, VVVC:FUSE_1A
- removed J5: 5V DC IN, VVVC:POWER_IN
Connections:
- JESP pad 19: +5V_SYS -> +5V_USB
Other:
- board text added: "GPIO22 PWM | M -> RX | B/C <- TX | USB 5V POWER"
- board text removed: "GPIO22 PWM | M -> RX | B/C <- TX"

Commit message: Add dual gang output volume control
Parts:
- added RV1: DUAL 10k AUDIO VOLUME, VVVC:VOLUME_DUAL_GANG, F.Cu at (85.0, 42.0)
Connections:
- J2 pad 1: LINE_OUT_L -> VOL_L
- J2 pad 2: LINE_OUT_R -> VOL_R
- J4 pad 1: LINE_OUT_L -> VOL_L
- J4 pad 2: LINE_OUT_R -> VOL_R
- U2 pad 3: LINE_OUT_L -> BUF_L
- U2 pad 4: LINE_OUT_R -> BUF_R
Other:
- board text added: "VOLUME"
Changed lines of the file:
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@@
   (net 9 "MIX_L")
   (net 10 "MIX_R")
-  (net 11 "LINE_OUT_L")
-  (net 12 "LINE_OUT_R")
-  (net 13 "HP_OUT_L")
-  (net 14 "HP_OUT_R")
-  (net 15 "RX_DIV")
-  (net 16 "PWM_F1")
-  (net 17 "PWM_F2")
+  (net 11 "BUF_L")
+  (net 12 "BUF_R")
+  (net 13 "VOL_L")
+  (net 14 "VOL_R")
+  (net 15 "LINE_OUT_L")
+  (net 16 "LINE_OUT_R")
+  (net 17 "HP_OUT_L")
+  (net 18 "HP_OUT_R")
+  (net 19 "RX_DIV")
+  (net 20 "PWM_F1")
+  (net 21 "PWM_F2")
 (footprint "VVVC:VIC_USER_PORT_EDGE" (layer "F.Cu") (at 50 4)
   (property "Reference" "J1" (at 0 -4 0) (layer "F.SilkS"))
@@
     (hide yes))
   (pad "1" thru_hole circle (at -1.27 0) (size 1.8 1.8) (drill 0.9) (layers "*.Cu" "*.Mask") (net 4 "VIC_RX"))
-  (pad "2" thru_hole circle (at 1.27 0) (size 1.8 1.8) (drill 0.9) (layers "*.Cu" "*.Mask") (net 15 "RX_DIV"))
+  (pad "2" thru_hole circle (at 1.27 0) (size 1.8 1.8) (drill 0.9) (layers "*.Cu" "*.Mask") (net 19 "RX_DIV"))
   (fp_rect (start -2.6 -1.5) (end 2.6 1.5) (stroke (width 0.2) (type default)) (fill none) (layer "F.SilkS"))
 )
@@
   (property "Value" "18k" (at 0 4 0) (layer "F.Fab")
     (hide yes))
-  (pad "1" thru_hole circle (at -1.27 0) (size 1.8 1.8) (drill 0.9) (layers "*.Cu" "*.Mask") (net 15 "RX_DIV"))
+  (pad "1" thru_hole circle (at -1.27 0) (size 1.8 1.8) (drill 0.9) (layers "*.Cu" "*.Mask") (net 19 "RX_DIV"))
   (pad "2" thru_hole circle (at 1.27 0) (size 1.8 1.8) (drill 0.9) (layers "*.Cu" "*.Mask") (net 1 "GND"))
   (fp_rect (start -2.6 -1.5) (end 2.6 1.5) (stroke (width 0.2) (type default)) (fill none) (layer "F.SilkS"))
@@
     (hide yes))
   (pad "1" thru_hole circle (at -1.27 0) (size 1.8 1.8) (drill 0.9) (layers "*.Cu" "*.Mask") (net 6 "PWM_AUDIO"))
-  (pad "2" thru_hole circle (at 1.27 0) (size 1.8 1.8) (drill 0.9) (layers "*.Cu" "*.Mask") (net 16 "PWM_F1"))
+  (pad "2" thru_hole circle (at 1.27 0) (size 1.8 1.8) (drill 0.9) (layers "*.Cu" "*.Mask") (net 20 "PWM_F1"))
   (fp_rect (start -2.6 -1.5) (end 2.6 1.5) (stroke (width 0.2) (type default)) (fill none) (layer "F.SilkS"))
 )
@@
   (property "Value" "4.7k" (at 0 4 0) (layer "F.Fab")
     (hide yes))
-  (pad "1" thru_hole circle (at -1.27 0) (size 1.8 1.8) (drill 0.9) (layers "*.Cu" "*.Mask") (net 16 "PWM_F1"))
-  (pad "2" thru_hole circle (at 1.27 0) (size 1.8 1.8) (drill 0.9) (layers "*.Cu" "*.Mask") (net 17 "PWM_F2"))
+  (pad "1" thru_hole circle (at -1.27 0) (size 1.8 1.8) (drill 0.9) (layers "*.Cu" "*.Mask") (net 20 "PWM_F1"))
+  (pad "2" thru_hole circle (at 1.27 0) (size 1.8 1.8) (drill 0.9) (layers "*.Cu" "*.Mask") (net 21 "PWM_F2"))
   (fp_rect (start -2.6 -1.5) (end 2.6 1.5) (stroke (width 0.2) (type default)) (fill none) (layer "F.SilkS"))
 )
@@
   (property "Value" "22nF" (at 0 4 0) (layer "F.Fab")
     (hide yes))
-  (pad "1" thru_hole circle (at -1.27 0) (size 1.8 1.8) (drill 0.9) (layers "*.Cu" "*.Mask") (net 16 "PWM_F1"))
+  (pad "1" thru_hole circle (at -1.27 0) (size 1.8 1.8) (drill 0.9) (layers "*.Cu" "*.Mask") (net 20 "PWM_F1"))
   (pad "2" thru_hole circle (at 1.27 0) (size 1.8 1.8) (drill 0.9) (layers "*.Cu" "*.Mask") (net 1 "GND"))
   (fp_rect (start -2.6 -1.5) (end 2.6 1.5) (stroke (width 0.2) (type default)) (fill none) (layer "F.SilkS"))
@@
   (property "Value" "4.7nF" (at 0 4 0) (layer "F.Fab")
     (hide yes))
-  (pad "1" thru_hole circle (at -1.27 0) (size 1.8 1.8) (drill 0.9) (layers "*.Cu" "*.Mask") (net 17 "PWM_F2"))
+  (pad "1" thru_hole circle (at -1.27 0) (size 1.8 1.8) (drill 0.9) (layers "*.Cu" "*.Mask") (net 21 "PWM_F2"))
   (pad "2" thru_hole circle (at 1.27 0) (size 1.8 1.8) (drill 0.9) (layers "*.Cu" "*.Mask") (net 1 "GND"))
   (fp_rect (start -2.6 -1.5) (end 2.6 1.5) (stroke (width 0.2) (type default)) (fill none) (layer "F.SilkS"))
@@
   (property "Value" "1uF FILM" (at 0 4 0) (layer "F.Fab")
     (hide yes))
-  (pad "1" thru_hole circle (at -1.27 0) (size 1.8 1.8) (drill 0.9) (layers "*.Cu" "*.Mask") (net 17 "PWM_F2"))
+  (pad "1" thru_hole circle (at -1.27 0) (size 1.8 1.8) (drill 0.9) (layers "*.Cu" "*.Mask") (net 21 "PWM_F2"))
   (pad "2" thru_hole circle (at 1.27 0) (size 1.8 1.8) (drill 0.9) (layers "*.Cu" "*.Mask") (net 9 "MIX_L"))
   (fp_rect (start -2.6 -1.5) (end 2.6 1.5) (stroke (width 0.2) (type default)) (fill none) (layer "F.SilkS"))
@@
   (property "Value" "10k" (at 0 4 0) (layer "F.Fab")
     (hide yes))
-  (pad "1" thru_hole circle (at -1.27 0) (size 1.8 1.8) (drill 0.9) (layers "*.Cu" "*.Mask") (net 17 "PWM_F2"))
+  (pad "1" thru_hole circle (at -1.27 0) (size 1.8 1.8) (drill 0.9) (layers "*.Cu" "*.Mask") (net 21 "PWM_F2"))
   (pad "2" thru_hole circle (at 1.27 0) (size 1.8 1.8) (drill 0.9) (layers "*.Cu" "*.Mask") (net 10 "MIX_R"))
   (fp_rect (start -2.6 -1.5) (end 2.6 1.5) (stroke (width 0.2) (type default)) (fill none) (layer "F.SilkS"))
@@
   (property "Value" "RCA OUT L/R" (at 0 4 0) (layer "F.Fab")
     (hide yes))
-  (pad "1" thru_hole circle (at -1.27 0) (size 1.8 1.8) (drill 0.9) (layers "*.Cu" "*.Mask") (net 11 "LINE_OUT_L"))
-  (pad "2" thru_hole circle (at 1.27 0) (size 1.8 1.8) (drill 0.9) (layers "*.Cu" "*.Mask") (net 12 "LINE_OUT_R"))
+  (pad "1" thru_hole circle (at -1.27 0) (size 1.8 1.8) (drill 0.9) (layers "*.Cu" "*.Mask") (net 13 "VOL_L"))
+  (pad "2" thru_hole circle (at 1.27 0) (size 1.8 1.8) (drill 0.9) (layers "*.Cu" "*.Mask") (net 14 "VOL_R"))
   (fp_rect (start -2.6 -1.5) (end 2.6 1.5) (stroke (width 0.2) (type default)) (fill none) (layer "F.SilkS"))
 )
@@
   (property "Value" "3.5mm TRS" (at 0 4 0) (layer "F.Fab")
     (hide yes))
-  (pad "1" thru_hole circle (at -2.54 0) (size 1.8 1.8) (drill 0.9) (layers "*.Cu" "*.Mask") (net 11 "LINE_OUT_L"))
-  (pad "2" thru_hole circle (at 0.0 0) (size 1.8 1.8) (drill 0.9) (layers "*.Cu" "*.Mask") (net 12 "LINE_OUT_R"))
+  (pad "1" thru_hole circle (at -2.54 0) (size 1.8 1.8) (drill 0.9) (layers "*.Cu" "*.Mask") (net 13 "VOL_L"))
+  (pad "2" thru_hole circle (at 0.0 0) (size 1.8 1.8) (drill 0.9) (layers "*.Cu" "*.Mask") (net 14 "VOL_R"))
   (pad "3" thru_hole circle (at 2.54 0) (size 1.8 1.8) (drill 0.9) (layers "*.Cu" "*.Mask") (net 1 "GND"))
   (fp_rect (start -3.9000000000000004 -1.5) (end 3.9000000000000004 1.5) (stroke (width 0.2) (type default)) (fill none) (layer "F.SilkS"))
@@
   (pad "1" thru_hole circle (at -6.35 0) (size 1.8 1.8) (drill 0.9) (layers "*.Cu" "*.Mask") (net 9 "MIX_L"))
   (pad "2" thru_hole circle (at -3.81 0) (size 1.8 1.8) (drill 0.9) (layers "*.Cu" "*.Mask") (net 10 "MIX_R"))
-  (pad "3" thru_hole circle (at -1.27 0) (size 1.8 1.8) (drill 0.9) (layers "*.Cu" "*.Mask") (net 11 "LINE_OUT_L"))
-  (pad "4" thru_hole circle (at 1.27 0) (size 1.8 1.8) (drill 0.9) (layers "*.Cu" "*.Mask") (net 12 "LINE_OUT_R"))
+  (pad "3" thru_hole circle (at -1.27 0) (size 1.8 1.8) (drill 0.9) (layers "*.Cu" "*.Mask") (net 11 "BUF_L"))
+  (pad "4" thru_hole circle (at 1.27 0) (size 1.8 1.8) (drill 0.9) (layers "*.Cu" "*.Mask") (net 12 "BUF_R"))
   (pad "5" thru_hole circle (at 3.81 0) (size 1.8 1.8) (drill 0.9) (layers "*.Cu" "*.Mask") (net 2 "+5V_USB"))
+  (pad "6" thru_hole circle (at 6.35 0) (size 1.8 1.8) (drill 0.9) (layers "*.Cu" "*.Mask") (net 1 "GND"))
+  (fp_rect (start -7.800000000000001 -1.5) (end 7.800000000000001 1.5) (stroke (width 0.2) (type default)) (fill none) (layer "F.SilkS"))
+)
+(footprint "VVVC:VOLUME_DUAL_GANG" (layer "F.Cu") (at 85 42)
+  (property "Reference" "RV1" (at 0 -4 0) (layer "F.SilkS"))
+  (property "Value" "DUAL 10k AUDIO VOLUME" (at 0 4 0) (layer "F.Fab")
+    (hide yes))
+  (pad "1" thru_hole circle (at -6.35 0) (size 1.8 1.8) (drill 0.9) (layers "*.Cu" "*.Mask") (net 11 "BUF_L"))
+  (pad "2" thru_hole circle (at -3.81 0) (size 1.8 1.8) (drill 0.9) (layers "*.Cu" "*.Mask") (net 13 "VOL_L"))
+  (pad "3" thru_hole circle (at -1.27 0) (size 1.8 1.8) (drill 0.9) (layers "*.Cu" "*.Mask") (net 1 "GND"))
+  (pad "4" thru_hole circle (at 1.27 0) (size 1.8 1.8) (drill 0.9) (layers "*.Cu" "*.Mask") (net 12 "BUF_R"))
+  (pad "5" thru_hole circle (at 3.81 0) (size 1.8 1.8) (drill 0.9) (layers "*.Cu" "*.Mask") (net 14 "VOL_R"))
   (pad "6" thru_hole circle (at 6.35 0) (size 1.8 1.8) (drill 0.9) (layers "*.Cu" "*.Mask") (net 1 "GND"))
   (fp_rect (start -7.800000000000001 -1.5) (end 7.800000000000001 1.5) (stroke (width 0.2) (type default)) (fill none) (layer "F.SilkS"))
@@
   (gr_text "VVVC USER-PORT AUDIO CARRIER" (at 50 75) (layer "F.SilkS") (effects (font (size 2 2) (thickness 0.3))))
   (gr_text "GPIO22 PWM  |  M -> RX  |  B/C <- TX  |  USB 5V POWER" (at 50 70) (layer "F.SilkS") (effects (font (size 1.2 1.2) (thickness 0.2))))
+  (gr_text "VOLUME" (at 85 38) (layer "F.SilkS") (effects (font (size 1.2 1.2) (thickness 0.2))))
   (gr_text "INSERT THIS EDGE INTO VIC USER PORT - COMPONENT SIDE UP" (at 50 12) (layer "F.SilkS") (effects (font (size 1.1 1.1) (thickness 0.18))))
   (gr_text "DRAFT - ROUTE AND VERIFY IN PCBNEW BEFORE FAB" (at 50 77) (layer "F.SilkS") (effects (font (size 1.2 1.2) (thickness 0.2))))
